File: kicad/interruptus/level_shifters.kicad_sch (KiCad schematic)
At the start: 8 parts, among them U6 SN74LVC1T45DBV, U7 SN74LVC1T45DBV, U8 SN74LVC1T45DBV, U9 SN74LVC1T45DBV

Commit message: small changes
Connections:
- net +3V3 is gone; now on net VCCA: U6.1 (VCCA), U7.1 (VCCA), U8.1 (VCCA), U9.1 (VCCA)
- net GND: now also U8.5 (DIR)
- net VCCA: now reaches U9.5 (DIR)
- net VCCA: now also U6.5 (DIR), U7.5 (DIR)
- net VBUS renamed VCCB
Other:
- moved on the sheet: R9, U9
