File: kicad/interruptus/untitled.kicad_sch (KiCad schematic)
At the start: 10 parts, among them J3 USB_B, U4 FT2232D, U5 74HC244, X1 6MHz

Commit message: small changes
Parts:
- removed J3: USB_B, symbol atmel-atdh1150usb-rescue:USB_B-Connector
- removed JP1: (unpopulated), symbol Jumper:Jumper_2_Open
- removed JP3: JTAG-A, symbol Connector_Generic:Conn_02x05_Odd_Even
- removed JP5: JTAG-X, symbol Connector_Generic:Conn_02x07_Odd_Even
- removed U5: 74HC244, symbol atmel-atdh1150usb-rescue:74HC244-74xx
- removed X1: 6MHz, symbol Device:Crystal_Small
- added C11, C12, C14: 100n, Capacitor_SMD:C_0603_1608Metric_Pad1.08x0.95mm_HandSolder, symbol Device:C
- added C13: 33n, Capacitor_SMD:C_0603_1608Metric_Pad1.08x0.95mm_HandSolder, symbol Device:C
- added D1, D2: 1N5819, Diode_SMD:Nexperia_CFP3_SOD-123W, symbol Diode:1N5819
- added P2: USB_C_Plug_USB2.0, Connector_USB:USB_C_Receptacle_G-Switch_GT-USB-7010ASV, symbol Connector:USB_C_Plug_USB2.0
- added Q1: IRLML6402, Package_TO_SOT_SMD:SOT-23, symbol Transistor_FET:IRLML6402
- added R4: 1k5, Resistor_SMD:R_0201_0603Metric_Pad0.64x0.40mm_HandSolder, symbol Device:R_Small
- added R5: 1k, Resistor_SMD:R_0201_0603Metric_Pad0.64x0.40mm_HandSolder, symbol Device:R_Small
- added R6: 1M, Resistor_SMD:R_0201_0603Metric_Pad0.64x0.40mm_HandSolder, symbol Device:R_Small
- added Y1: 6Mhz, Crystal:Resonator_Murata_CSTLSxxxX-3Pin_W5.5mm_H3.0mm, symbol Device:Resonator
- R1, R2: footprint (none) -> Resistor_SMD:R_0201_0603Metric_Pad0.64x0.40mm_HandSolder
- R3: value 10kR -> 470R; footprint (none) -> Resistor_SMD:R_0201_0603Metric_Pad0.64x0.40mm_HandSolder
Connections:
- net TCK_3V3 is gone; now on net TCK: U4.24 (ADBUS0)
- net TDI_3V3 is gone; now on net TDI: U4.23 (ADBUS1)
- net TDO_3V3 is gone; now on net TDO: U4.22 (ADBUS2)
- net TMS_3V3 is gone; now on net TMS: U4.21 (ADBUS3)
- net +5V: now also C12.1, D2.1 (K), Q1.3 (D)
- net GND: now also U4.18 (GND), U4.25 (GND), U4.34 (GND), U4.45 (AGND), U4.47 (TEST), U4.9 (GND), C11.2, C13.1, C14.1, P2.A1 (GND), P2.A12 (GND), P2.B1 (GND), P2.B12 (GND), P2.S1 (SHIELD), Y1.2; no longer R3.1
- net VBUS: now also D1.2 (A), P2.A4 (VBUS), P2.A9 (VBUS), P2.B4 (VBUS), P2.B9 (VBUS)
- net at R1.1: now also U4.8 (USBDM); no longer U4.7 (USBDP)
- net at R1.2: now also P2.A7 (D-)
- net at R3.2: now also U4.46 (AVCC), C14.2
- net VCCUSB: now reaches U4.14 (VCCIOA)
- net VCCUSB: now also R3.1, U4.3 (VCC), U4.31 (VCCIOB), U4.4 (~{RESET}), U4.42 (VCC), C11.1, D1.1 (K), Q1.2 (S)
- net at U4.41 (~{PWREN}): now also R5.1
- net at U4.43 (XTIN): now also R6.1, Y1.1
- net at U4.44 (XTOUT): now also R6.2, Y1.3
- net at U4.5 (~{RSTOUT}): now also R4.1
- net at U4.6 (3V3OUT): now also C13.2
- net at R2.1: now also U4.7 (USBDP), R4.2; no longer U4.8 (USBDM)
- net at R2.2: now also P2.A6 (D+)
- net 2~{OE}: no longer names the net of U4.13 (ACBUS1)
- net ADBUS5: no longer names the net of U4.19 (ADBUS5)
- net ADBUS6: no longer names the net of U4.17 (ADBUS6)
- net ADBUS7: no longer names the net of U4.16 (ADBUS7)
- net BDBUS0: no longer names the net of U4.40 (BDBUS0)
- net BDBUS1: no longer names the net of U4.39 (BDBUS1)
- net BDBUS2: no longer names the net of U4.38 (BDBUS2)
- net BDBUS3: no longer names the net of U4.37 (BDBUS3)
- net BDBUS4: no longer names the net of U4.36 (BDBUS4)
- net BDBUS5: no longer names the net of U4.35 (BDBUS5)
- net BDBUS6: no longer names the net of U4.33 (BDBUS6)
- net BDBUS7: no longer names the net of U4.32 (BDBUS7)
- new net: C12.2, Q1.1 (G), R5.2
- new net B_VCC: D2.2 (A)
- no-connect marks 17 -> 27
Other:
- removed sheet level_shifters
- note added: "Soft Start Circuit"
- note removed: "Incomplete..."
- note removed: "Note: The user manual states, that the TWI interface is broken on this board!"
- note removed: "to U1"
- note removed: "to U2"
- note removed: "to U5"
- note removed: "to U7"
- moved on the sheet: R1, R2, U4

Commit message: new usb connector, and other changes
Parts:
- removed P2: USB_C_Plug_USB2.0, Connector_USB:USB_C_Receptacle_G-Switch_GT-USB-7010ASV, symbol Connector:USB_C_Plug_USB2.0
- removed Q1: IRLML6402, Package_TO_SOT_SMD:SOT-23, symbol Transistor_FET:IRLML6402
- removed R6: 1M, Resistor_SMD:R_0201_0603Metric_Pad0.64x0.40mm_HandSolder, symbol Device:R_Small
- removed Y1: 6Mhz, Crystal:Resonator_Murata_CSTLSxxxX-3Pin_W5.5mm_H3.0mm, symbol Device:Resonator
- added J3: USB4110GFA, USB4110GFA:GCT_USB4110GFA, symbol USB4110GFA:USB4110GFA
- added R7: 5k1, Resistor_SMD:R_0201_0603Metric_Pad0.64x0.40mm_HandSolder, symbol Device:R_Small
- added Y1: 6 MHz, symbol Device:Crystal
- C11, C12: value 100n -> 27p
- R5: value 1k -> 5k1
Connections:
- net +5V: now also D1.1 (K), R3.1, U4.14 (VCCIOA), U4.3 (VCC), U4.31 (VCCIOB), U4.42 (VCC); no longer C12.1
- net GND: now also C11.1, C12.1, R5.1, J3.A1/B12 (GND), J3.B1/A12 (GND), J3.S1 (GND), J3.S2 (GND), J3.S3 (GND), J3.S4 (GND), R7.1; no longer C11.2
- net VBUS: now also J3.A4/B9 (VBUS), J3.B4/A9 (VBUS)
- net VCCUSB: no longer C11.1, D1.1 (K), R3.1, U4.14 (VCCIOA), U4.3 (VCC), U4.31 (VCCIOB), U4.42 (VCC)
- net at U4.43 (XTIN): now also C11.2, Y1.1
- net at U4.44 (XTOUT): now also C12.2, Y1.2
- net at U4.41 (~{PWREN}): no longer R5.1
- net at R5.2: now also J3.A5 (CC1); no longer C12.2
- net at R1.2: now also J3.A7 (DN1), J3.B7 (DN2)
- net at R2.2: now also J3.A6 (DP1), J3.B6 (DP2)
- net RESET_FTDI: now reaches U4.13 (ACBUS1)
- net GCLR_FTDI: now reaches U4.15 (ACBUS0)
- new net: J3.B5 (CC2), R7.2
- no-connect marks 27 -> 23
Other:
- note removed: "Soft Start Circuit"
- moved on the sheet: D1
