File: kicad/interruptus/interruptus.kicad_pcb (KiCad board)
At the start: 4 copper layers, 75.5 x 100 mm, 31 parts, among them IC1 ATF1508AS-7JX84, J1 Conn_02x16_Counter_Clockwise, J2 Conn_01x03_Pin, P1 C96ABC, P2 USB_C_Plug_USB2.0, Q1 IRLML6402, U1 LTC6905xS5-133, U2 TPS7A2033, U4 FT2232D, Y1 6Mhz

Commit message: rev 5
Parts:
- removed C10, C9: 1u, Capacitor_SMD:C_0603_1608Metric_Pad1.08x0.95mm_HandSolder
- removed C11, C12, C14: 100n, Capacitor_SMD:C_0603_1608Metric_Pad1.08x0.95mm_HandSolder
- removed C13: 33n, Capacitor_SMD:C_0603_1608Metric_Pad1.08x0.95mm_HandSolder
- removed D1, D2: 1N5819, Diode_SMD:Nexperia_CFP3_SOD-123W
- removed IC1: ATF1508AS-7JX84, Package_LCC:PLCC-84
- removed P2: USB_C_Plug_USB2.0, Connector_USB:USB_C_Receptacle_G-Switch_GT-USB-7010ASV
- added D3: LED, LED_SMD:LED_0402_1005Metric, F.Cu at (138.2, 64.0)
- added D4: LED, LED_SMD:LED_0402_1005Metric, F.Cu at (138.2, 69.1)
- added D5: LED, LED_SMD:LED_0402_1005Metric, F.Cu at (138.2, 73.5)
- added J3: USB4110GFA, Library:USB_C_Receptacle_GCT_USB4110, B.Cu at (145.8, 123.0)
- added Q2: 2N7002, Package_TO_SOT_SMD:SOT-23, B.Cu at (102.9, 123.5)
- added R10: 1k5, Resistor_SMD:R_0201_0603Metric_Pad0.64x0.40mm_HandSolder, B.Cu at (125.5, 134.2)
- added R11: 470R, Resistor_SMD:R_0201_0603Metric_Pad0.64x0.40mm_HandSolder, B.Cu at (124.0, 129.0)
- added R12: 5k1, Resistor_SMD:R_0201_0603Metric_Pad0.64x0.40mm_HandSolder, F.Cu at (142.0, 64.0)
- added R13: 5k1, Resistor_SMD:R_0201_0603Metric_Pad0.64x0.40mm_HandSolder, F.Cu at (142.0, 69.0)
- added R14: 5k1, Resistor_SMD:R_0201_0603Metric_Pad0.64x0.40mm_HandSolder, F.Cu at (142.0, 73.5)
- added R15: 2k2, Resistor_SMD:R_0201_0603Metric_Pad0.64x0.40mm_HandSolder, B.Cu at (96.2, 137.0)
- added R16: 10k, Resistor_SMD:R_0201_0603Metric_Pad0.64x0.40mm_HandSolder, B.Cu at (96.8, 139.8)
- added R6: 5k1, Resistor_SMD:R_0201_0603Metric_Pad0.64x0.40mm_HandSolder, B.Cu at (140.0, 115.0)
- added R7: 5k1, Resistor_SMD:R_0201_0603Metric_Pad0.64x0.40mm_HandSolder, B.Cu at (139.0, 128.5)
- added R8: 27R, Resistor_SMD:R_0201_0603Metric_Pad0.64x0.40mm_HandSolder, B.Cu at (139.4, 123.5)
- added R9: 27R, Resistor_SMD:R_0201_0603Metric_Pad0.64x0.40mm_HandSolder, B.Cu at (139.4, 122.5)
- added U3: TPS7A2033, Package_TO_SOT_SMD:SOT-23-5, B.Cu at (125.1, 61.5)
- added U5: 93CxxB, Package_SO:SOIC-8_3.9x4.9mm_P1.27mm, B.Cu at (103.2, 137.2)
- added U6: MAX40200AUK, Package_TO_SOT_SMD:SOT-23-5, B.Cu at (87.5, 137.0)
- added U7: MAX40200AUK, Package_TO_SOT_SMD:SOT-23-5, B.Cu at (134.2, 121.5)
- C1, C3, C8, U4: moved to B.Cu
- C2, C4: value 100n -> 1u; moved to B.Cu
- C5, C6: value 100n -> 8p; moved to B.Cu
- C7: value 100n -> 33n; moved to B.Cu
- J1: value Conn_02x16_Counter_Clockwise -> Conn_01x03_Pin; footprint Connector_PinHeader_2.54mm:PinHeader_2x16_P2.54mm_Vertical -> Connector_PinHeader_2.54mm:PinHeader_1x03_P2.54mm_Vertical
- J2: value Conn_01x03_Pin -> Conn_02x08_Counter_Clockwise; footprint Connector_PinHeader_2.54mm:PinHeader_1x03_P2.54mm_Vertical -> Connector_PinHeader_2.54mm:PinHeader_2x08_P2.54mm_Vertical
- Q1: value IRLML6402 -> 2N7002; moved to B.Cu
- R1, R2: value 27R -> 5k1; moved to B.Cu
- R3: value 470R -> 5k1; moved to B.Cu
- R4: value 1k5 -> 5k1; moved to B.Cu
- R5: value 1k -> 0R; moved to B.Cu
- U1: value LTC6905xS5-133 -> ATF1508AS-7JX84; footprint Package_TO_SOT_SMD:TSOT-23-5 -> Package_LCC:PLCC-84_THT-Socket
- U2: value TPS7A2033 -> LTC6905xS5-100; footprint Package_TO_SOT_SMD:SOT-23-5 -> Package_TO_SOT_SMD:TSOT-23-5; moved to B.Cu
- Y1: value 6Mhz -> 6 MHz; footprint Crystal:Resonator_Murata_CSTLSxxxX-3Pin_W5.5mm_H3.0mm -> Library:Crystal_SMD_8045-2Pin_8.0x4.5mm_HandSoldering; moved to B.Cu
- moved J1 78.5 mm to (111.1, 60.0), turned to 0 degrees
- moved C7 74.7 mm to (126.6, 130.8), turned to 180 degrees
- moved C8 70.5 mm to (126.6, 129.0), turned to 180 degrees
- moved C1 54.9 mm to (92.2, 73.8), turned to 180 degrees
- moved C5 54.0 mm to (111.0, 125.0), turned to 90 degrees
- moved R5 52.5 mm to (118.8, 71.0), turned to -90 degrees
- moved C6 47.8 mm to (125.0, 125.0), turned to 90 degrees
- moved Q1 47.4 mm to (140.3, 82.6), turned to 90 degrees
- moved R3 44.5 mm to (143.0, 83.5), turned to -90 degrees
- moved C2 40.8 mm to (129.6, 60.5)
- moved R2 39.6 mm to (98.1, 122.0)
- moved U2 37.1 mm to (119.7, 66.1), turned to -90 degrees
- moved C4 36.9 mm to (120.2, 60.5), turned to 180 degrees
- moved U1 32.9 mm to (112.7, 78.5), turned to 0 degrees
- moved R1 32.9 mm to (140.2, 78.8), turned to -90 degrees
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Connections:
- C1 pad 1: +3.3V -> +5V
- C2 pad 1: VCC -> GND
- C2 pad 2: GND -> +5V
- C3 pad 1: VCC -> +3.3V
- C4 pad 1: VCC -> +3.3V
- C5 pad 1: VCC -> GND
- C5 pad 2: GND -> Net-(U4-XTIN)
- C6 pad 1: VCC -> GND
- C6 pad 2: GND -> Net-(U4-XTOUT)
- C7 pad 1: VCC -> GND
- C7 pad 2: GND -> Net-(U4-3V3OUT)
- C8 pad 1: VCC -> GND
- C8 pad 2: GND -> Net-(U4-AVCC)
- J1 pad 1: GND -> +3.3V
- J1 pad 2: /I/OE1 -> Net-(J1-Pin_2)
- J1 pad 3: /I/GCLR -> GND
- J2 pad 1: VCC -> /TDI
- J2 pad 2: Net-(J2-Pin_2) -> /TDO
- J2 pad 3: GND -> /TCK
- P1 pad b10: unconnected-(P1-10B-Padb10) -> B_D12
- P1 pad b11: unconnected-(P1-11B-Padb11) -> B_D13
- P1 pad b12: unconnected-(P1-12B-Padb12) -> B_D14
- P1 pad b13: unconnected-(P1-13B-Padb13) -> B_D15
- P1 pad b22: unconnected-(P1-22B-Padb22) -> B_ / SXTAK
- P1 pad b24: unconnected-(P1-24B-Padb24) -> B_ / SXTRQ
- P1 pad b28: unconnected-(P1-28B-Padb28) -> B_ / DS0
- P1 pad b29: unconnected-(P1-29B-Padb29) -> B_ / DS1
- P1 pad b6: unconnected-(P1-6B-Padb6) -> B_D8
- P1 pad b7: unconnected-(P1-7B-Padb7) -> B_D9
- P1 pad b8: unconnected-(P1-8B-Padb8) -> B_D10
- P1 pad b9: unconnected-(P1-9B-Padb9) -> B_D11
- Q1 pad 1: Net-(Q1-G) -> /GCLR_FTDI
- Q1 pad 2: /JTAG-Interface/VCCUSB -> GND
- Q1 pad 3: VCC -> /I/GCLR
- R1 pad 1: Net-(U4-USBDM) -> +5V
- R1 pad 2: Net-(P2-D-) -> /I/GCLR
- R2 pad 1: Net-(U4-USBDP) -> +5V
- R2 pad 2: Net-(P2-D+) -> /B_/RESET
- R3 pad 1: /JTAG-Interface/VCCUSB -> /GCLR_FTDI
- R3 pad 2: Net-(U4-AVCC) -> GND
- R4 pad 1: Net-(U4-~{RSTOUT}) -> /RESET_FTDI
- R4 pad 2: Net-(U4-USBDP) -> GND
- R5 pad 1: Net-(U4-~{PWREN}) -> Net-(U2-OUT)
- R5 pad 2: Net-(Q1-G) -> /GCLK1
- U1 pad 1: +3.3V -> /I/GCLR
- U1 pad 2: GND -> /I/OE2/GCLK2
- U1 pad 3: unconnected-(U1-OE-Pad3) -> +5V
- U1 pad 4: Net-(J2-Pin_2) -> B_D5
- U1 pad 5: /GCLK1 -> B_D6
- U2 pad 1: VCC -> +3.3V
- U2 pad 3: VCC -> unconnected-(U2-OE-Pad3)
- U2 pad 4: (no net) -> Net-(J1-Pin_2)
- U2 pad 5: +3.3V -> Net-(U2-OUT)
- U4 pad 1: unconnected-(U4-EECLK-Pad1) -> Net-(U4-EECLK)
- U4 pad 13: unconnected-(U4-ACBUS1-Pad13) -> /RESET_FTDI
- U4 pad 14: /JTAG-Interface/VCCUSB -> +5V
- U4 pad 15: unconnected-(U4-ACBUS0-Pad15) -> /GCLR_FTDI
- U4 pad 2: unconnected-(U4-EEDATA-Pad2) -> Net-(U4-EEDATA)
- U4 pad 26: unconnected-(U4-SI/WUB-Pad26) -> /I/O/GCLK3
- U4 pad 27: unconnected-(U4-BCBUS3-Pad27) -> /I/O/PD2
- U4 pad 28: unconnected-(U4-BCBUS2-Pad28) -> /I/O/PD1
- U4 pad 29: unconnected-(U4-BCBUS1-Pad29) -> /I/OE2/GCLK2
- U4 pad 3: /JTAG-Interface/VCCUSB -> +5V
- U4 pad 30: unconnected-(U4-BCBUS0-Pad30) -> /I/OE1
- U4 pad 31: /JTAG-Interface/VCCUSB -> +5V
- U4 pad 32: unconnected-(U4-BDBUS7-Pad32) -> B_D7
- U4 pad 33: unconnected-(U4-BDBUS6-Pad33) -> B_D6
- U4 pad 35: unconnected-(U4-BDBUS5-Pad35) -> B_D5
- U4 pad 36: unconnected-(U4-BDBUS4-Pad36) -> B_D4
- U4 pad 37: unconnected-(U4-BDBUS3-Pad37) -> B_D3
- U4 pad 38: unconnected-(U4-BDBUS2-Pad38) -> B_D2
- U4 pad 39: unconnected-(U4-BDBUS1-Pad39) -> B_D1
- U4 pad 4: /JTAG-Interface/VCCUSB -> +5V
- U4 pad 40: unconnected-(U4-BDBUS0-Pad40) -> B_D0
- U4 pad 41: Net-(U4-~{PWREN}) -> unconnected-(U4-~{PWREN}-Pad41)
- U4 pad 42: /JTAG-Interface/VCCUSB -> +5V
- U4 pad 48: unconnected-(U4-EECS-Pad48) -> Net-(U4-EECS)
- U4 pad 7: Net-(U4-USBDP) -> /JTAG-Interface/FTDI_USB_DATA+
- U4 pad 8: Net-(U4-USBDM) -> /JTAG-Interface/FTDI_USB_DATA-
- Y1 pad 2: GND -> Net-(U4-XTOUT)
Routing:
- net GND: track 367.9 -> 54.0 mm, vias 1 -> 33
- net VCC: track 258.7 -> 0.00 mm, vias 2 -> 0
- net /B_/RESET: track 17.9 -> 113.9 mm, vias 0 -> 1
- net /GCLR_FTDI: track 0.00 -> 79.2 mm, vias 0 -> 2
- net /IO_6: track 76.0 -> 0.00 mm, vias 1 -> 0
- net B_D10: track 0.00 -> 76.0 mm, vias 0 -> 2
- net /IO_4: track 74.6 -> 0.00 mm, vias 1 -> 0
- net /IO_7: track 74.1 -> 0.00 mm, vias 1 -> 0
- net /GCLK1: track 82.1 -> 8.49 mm, vias 2 -> 0
- net /IO_5: track 73.0 -> 0.00 mm, vias 1 -> 0
- net B_D9: track 0.00 -> 72.4 mm, vias 0 -> 1
- net /IO_26: track 71.7 -> 0.00 mm, vias 1 -> 0
- net /IO_25: track 70.2 -> 0.00 mm, vias 1 -> 0
- net B_ / DS1: track 0.00 -> 67.9 mm, vias 0 -> 1
- net /IO_28: track 66.8 -> 0.00 mm, vias 1 -> 0
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- added copper zone on In1.Cu, net +5V
- added copper zone on F.Cu, net GND
- added copper zone on In2.Cu, net GND
- removed copper zone on In1.Cu, net GND
- removed copper zone on In2.Cu, net VCC

Commit message: rev 8
Parts:
- removed D4, D5: LED, LED_SMD:LED_0402_1005Metric
- removed J2: Conn_02x08_Counter_Clockwise, Connector_PinHeader_2.54mm:PinHeader_2x08_P2.54mm_Vertical
- added D1: LED, LED_SMD:LED_0603_1608Metric_Pad1.05x0.95mm_HandSolder, F.Cu at (170.7, 46.9)
- added D2: LED, LED_SMD:LED_0603_1608Metric_Pad1.05x0.95mm_HandSolder, F.Cu at (170.7, 52.0)
- added G***: LOGO, KiCad:logo, F.Cu at (122.5, 128.3)
- added J4: Conn_02x20_Counter_Clockwise, Connector_PinHeader_2.54mm:PinHeader_2x20_P2.54mm_Vertical, F.Cu at (165.6, 69.8)
- added R17: 10k, Resistor_SMD:R_0603_1608Metric_Pad0.98x0.95mm_HandSolder, B.Cu at (148.7, 131.8)
- D3: footprint LED_SMD:LED_0402_1005Metric -> LED_SMD:LED_0603_1608Metric_Pad1.05x0.95mm_HandSolder
- R1, R10, R11, R15, R16, R2, R3, R4, R5, R6, R7, R8, R9: footprint Resistor_SMD:R_0201_0603Metric_Pad0.64x0.40mm_HandSolder -> Resistor_SMD:R_0603_1608Metric_Pad0.98x0.95mm_HandSolder
- R12, R13, R14: footprint Resistor_SMD:R_0201_0603Metric_Pad0.64x0.40mm_HandSolder -> Resistor_SMD:R_0603_1608Metric_Pad0.98x0.95mm_HandSolder; moved to B.Cu
- moved D3 33.4 mm to (170.7, 56.2), turned to 180 degrees
- moved U7 29.7 mm to (163.7, 125.7), turned to 90 degrees
- moved R12 29.2 mm to (165.6, 46.9)
- moved R13 29.2 mm to (165.6, 51.9)
- moved R14 28.3 mm to (164.4, 56.3), turned to 0 degrees
- moved R6 27.9 mm to (162.8, 131.0), turned to -90 degrees
- moved J3 27.1 mm to (170.3, 134.6)
- moved R7 25.8 mm to (162.8, 138.3)
- moved R8 24.0 mm to (160.1, 135.6)
- moved R9 23.5 mm to (160.1, 133.6)
- moved R10 17.3 mm to (142.7, 132.6), turned to 0 degrees
- moved C8 16.2 mm to (142.7, 127.4)
- moved C7 16.2 mm to (142.7, 129.6)
- moved C5 15.8 mm to (126.7, 123.3)
- moved R11 15.0 mm to (138.9, 128.1)
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Connections:
- J3 pad B4/A9: (no net) -> /JTAG-Interface/VBUS
- R12 pad 2: Net-(D3-A) -> Net-(D1-A)
- R14 pad 2: Net-(D5-A) -> Net-(D3-A)
- U4 pad 4: +5V -> Net-(U4-~{RESET})
Routing:
- net /B_/IRQ1: track 19.9 -> 181.8 mm, vias 0 -> 2
- net /B_/RD: track 33.2 -> 183.0 mm, vias 0 -> 1
- net /B_/IRQ4: track 16.1 -> 147.7 mm, vias 0 -> 4
- net /B_/IRQ2: track 19.2 -> 132.2 mm, vias 0 -> 2
- net B_D5: track 88.2 -> 184.8 mm, vias 3 -> 5
- net B_VCC: track 8.64 -> 99.0 mm, vias 0 -> 1
- net /B_/IRQ3: track 16.0 -> 96.7 mm, vias 0 -> 1
- net /B_/WR: track 26.9 -> 99.4 mm, vias 0 -> 1
- net /B_/IRQ0: track 19.7 -> 90.9 mm
- net B_D3: track 96.6 -> 165.7 mm
- net B_D1: track 90.8 -> 158.9 mm
- net /I/O/GCLK3: track 114.1 -> 178.1 mm, vias 3 -> 5
- net B_D7: track 93.4 -> 155.8 mm, vias 2 -> 3
- net B_A5: track 67.2 -> 125.6 mm, vias 1 -> 3
- net B_D4: track 91.8 -> 144.8 mm, vias 4 -> 3
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Other:
- board size 75.5 x 100 mm -> 100 x 100 mm
- board text added: "1"
- board text added: "2"
- board text added: "3"
- board text added: "3.3V"
- board text added: "5V"
- board text added: "A0"
- board text added: "A1"
- board text added: "A2"
- board text added: "A3"
- board text added: "A4"
- board text added: "A5"
- board text added: "A6"
- board text added: "A7"
- board text added: "A8"
- board text added: "D0"
- board text added: "D1"
- board text added: "D2"
- board text added: "D3"
- board text added: "D4"
- board text added: "D5"
- board text added: "D6"
- board text added: "D7"
- board text added: "GCLK2"
- board text added: "GCLK3"
- board text added: "GCLR"
- board text added: "GND"
- board text added: "IRQ0"
- board text added: "IRQ1"
- board text added: "IRQ2"
- board text added: "IRQ3"
- board text added: "IRQ4"
- board text added: "OE1"
- board text added: "PD1"
- board text added: "PD2"
- board text added: "RD"
- board text added: "Rev. 8"
- board text added: "TCK"
- board text added: "TDI"
- board text added: "TDO"
- board text added: "TMS"
- board text added: "VCC"
- board text added: "WR"
- board text added: "https://github.com/parceval/interrruptus"
