File: kicad/interruptus/interruptus.kicad_sch (KiCad schematic)
At the start: 16 parts, among them IC1 ATF1508AS-7JX84, J1 Conn_02x16_Counter_Clockwise, J2 Conn_01x03_Pin, P1 C96ABC, U1 LTC6905xS5-133

Commit message: small changes
Parts:
- removed U1: LTC6905xS5-133, Package_TO_SOT_SMD:TSOT-23-5, symbol Oscillator:LTC6905xS5-133
- added U3: LTC6905xS5-100, Package_TO_SOT_SMD:TSOT-23-5, symbol Oscillator:LTC6905xS5-100
- C1, C10, C2, C3, C4, C5, C6, C7, C8, C9: footprint (none) -> Capacitor_SMD:C_0603_1608Metric_Pad1.08x0.95mm_HandSolder
- IC1: footprint PLCC127P3023X3023X457-84N -> Package_LCC:PLCC-84
- J1: footprint (none) -> Connector_PinHeader_2.54mm:PinHeader_2x16_P2.54mm_Vertical
- J2: footprint (none) -> Connector_PinHeader_2.54mm:PinHeader_1x03_P2.54mm_Vertical
- P1: footprint 01N8VEM:C96ABCM-RA -> Connector_DIN:DIN41612_R_3x32_Female_Horizontal_THT; symbol PIC-007-rescue:C96ABC-00N8VEM1 -> Interruptus_Library:C96ABC-00N8VEM1
- U2: value ~ -> TPS7A2033; footprint (none) -> Package_TO_SOT_SMD:SOT-23-5
Connections:
- net 3V3 is gone; now on net +3.3V: C1.1, C9.1, U2.5 (OUT)
- net BAI/O: now also P1.a12 (12A), P1.a17 (17A); no longer P1.A12 (12A), P1.A17 (17A)
- net B_/DREQ: now also P1.b23 (23B); no longer P1.B23 (23B)
- net B_/INT: now also P1.c21 (21C); no longer P1.C21 (21C)
- net B_/INTA: now also P1.b25 (25B); no longer P1.B25 (25B)
- net B_/IORQ: now also P1.a27 (27A); no longer P1.A27 (27A)
- net B_/IRQ0: now also P1.b21 (21B); no longer P1.B21 (21B)
- net B_/IRQ1: now also P1.b20 (20B); no longer P1.B20 (20B)
- net B_/IRQ2: now also P1.b19 (19B); no longer P1.B19 (19B)
- net B_/IRQ3: now also P1.b18 (18B); no longer P1.B18 (18B)
- net B_/IRQ4: now also P1.b17 (17B); no longer P1.B17 (17B)
- net B_/IRQ5: now also P1.b16 (16B); no longer P1.B16 (16B)
- net B_/IRQ6: now also P1.b15 (15B); no longer P1.B15 (15B)
- net B_/IRQ7: now also P1.b14 (14B); no longer P1.B14 (14B)
- net B_/M1: now also P1.a20 (20A); no longer P1.A20 (20A)
- net B_/RD: now also P1.c24 (24C); no longer P1.C24 (24C)
- net B_/RESET: now also P1.c31 (31C); no longer P1.C31 (31C)
- net B_/RESOUT: now also P1.c26 (26C); no longer P1.C26 (26C)
- net B_/WR: now also P1.c22 (22C); no longer P1.C22 (22C)
- net B_A0: now also P1.c5 (5C); no longer P1.C5 (5C)
- net B_A1: now also P1.c7 (7C); no longer P1.C7 (7C)
- net B_A10: now also P1.c18 (18C); no longer P1.C18 (18C)
- net B_A11: now also P1.c17 (17C); no longer P1.C17 (17C)
- net B_A12: now also P1.c27 (27C); no longer P1.C27 (27C)
- net B_A13: now also P1.a29 (29A); no longer P1.A29 (29A)
- net B_A14: now also P1.a18 (18A)
- net B_A15: now also P1.a28 (28A)
- net B_A2: now also P1.a6 (6A); no longer P1.A6 (6A)
- net B_A3: now also P1.c6 (6C); no longer P1.C6 (6C)
- net B_A4: now also P1.a7 (7A); no longer P1.A7 (7A)
- net B_A5: now also P1.a8 (8A); no longer P1.A8 (8A)
- net B_A6: now also P1.a9 (9A); no longer P1.A9 (9A)
- net B_A7: now also P1.c9 (9C); no longer P1.C9 (9C)
- net B_A8: now also P1.c8 (8C); no longer P1.C8 (8C)
- net B_A9: now also P1.a30 (30A); no longer P1.A30 (30A)
- net B_D0: now also P1.c2 (2C); no longer P1.C2 (2C)
- net B_D1: now also P1.c14 (14C); no longer P1.C14 (14C)
- net B_D2: now also P1.c4 (4C); no longer P1.C4 (4C)
- net B_D3: now also P1.a4 (4A); no longer P1.A4 (4A)
- net B_D4: now also P1.a5 (5A); no longer P1.A5 (5A)
- net B_D5: now also P1.a2 (2A); no longer P1.A2 (2A)
- net B_D6: now also P1.a3 (3A); no longer P1.A3 (3A)
- net B_D7: now also P1.c3 (3C); no longer P1.C3 (3C)
- net B_VBAT: now also P1.a24 (24A); no longer P1.A24 (24A)
- net GCLK1: now also J1.6 (Pin_6), U3.5 (OUT)
- net GND: now also P1.a32 (32A), P1.b32 (32B), P1.c32 (32C), U3.2 (GND); no longer P1.A32 (32A), P1.B32 (32B), P1.C32 (32C)
- net IEI/O: now also P1.c11 (11C), P1.c16 (16C); no longer P1.C11 (11C), P1.C16 (16C)
- net TCK: now also J1.23 (Pin_23)
- net TDI: now also J1.21 (Pin_21)
- net TDO: now also J1.22 (Pin_22)
- net TMS: now also J1.24 (Pin_24)
- net at J2.2 (Pin_2): now also U3.4 (DIV)
- net I/OE1: now reaches J1.2 (Pin_2)
- net I/OE1: now also IC1.84 (INPUT/OE1)
- net I/GCLR: now reaches J1.3 (Pin_3)
- net I/GCLR: now also IC1.1 (INPUT/GCLR)
- net +3.3V: now reaches J1.31 (Pin_31)
- net +3.3V: now also U3.1 (VDD)
- net I/O/GCLK3: now reaches J1.4 (Pin_4)
- net I/O/GCLK3: now also IC1.81 (I/O/GCLK3)
- net I/O/PD1: now reaches IC1.12 (I/O/PD1)
- net I/O/PD1: now also J1.8 (Pin_8)
- net I/OE2/GCLK2: now reaches IC1.2 (INPUT/OE2/GCLK2)
- net I/OE2/GCLK2: now also J1.5 (Pin_5)
- net I/O/PD2: now reaches IC1.45 (I/O/PD2)
- net I/O/PD2: now also J1.7 (Pin_7)
- net IO_33 renamed B_A19
- net B_A19: now also P1.a14 (14A); no longer J1.8 (Pin_8)
- net IO_34 renamed B_A18
- net B_A18: now also P1.c13 (13C); no longer J1.7 (Pin_7)
- net IO_35 renamed B_A17
- net B_A17: now also P1.c12 (12C); no longer J1.6 (Pin_6)
- net IO_36 renamed B_A16
- net B_A16: now also P1.c10 (10C); no longer J1.5 (Pin_5)
- net VCC renamed +5V
- net +5V: no longer P1.A1 (1A), P1.B1 (1B), P1.C1 (1C)
- new net B_VCC: P1.a1 (1A), P1.b1 (1B), P1.c1 (1C)
- no-connect marks 47 -> 48
Other:
- sheet JTAG-Interface ports: added TCK, TDI, TDO, TMS; removed none
- note added: "133 MHz Clock Generator"
- note added: "3,3V Voltage Regulator"
- moved on the sheet: C1, C10, C9, J1, J2, U2

Commit message: new usb connector, and other changes
Parts:
- removed C3, C4, C5, C6, C7, C8: 100n, Capacitor_SMD:C_0603_1608Metric_Pad1.08x0.95mm_HandSolder, symbol Device:C
- added Q1, Q2: 2N7002, Package_TO_SOT_SMD:SOT-23, symbol Transistor_FET:2N7002
- added R6, R8: 5k1, symbol Device:R
Connections:
- net +5V: now also R6.1, R8.1
- net B_/RESET: now also Q2.3 (D), R8.2
- net GCLK1: no longer J1.6 (Pin_6)
- net GND: now also Q1.2 (S), Q2.2 (S)
- net IO_30: now also J1.16 (Pin_16); no longer J1.11 (Pin_11)
- net I/GCLR: now also J1.12 (Pin_12), Q1.3 (D), R6.2; no longer J1.3 (Pin_3)
- net I/OE1: now also J1.11 (Pin_11); no longer J1.2 (Pin_2)
- net I/OE2/GCLK2: now also J1.14 (Pin_14); no longer J1.5 (Pin_5)
- net I/O/GCLK3: now also J1.13 (Pin_13); no longer J1.4 (Pin_4)
- net I/O/PD2: now also J1.15 (Pin_15); no longer J1.7 (Pin_7)
- net TCK: now also J1.19 (Pin_19); no longer J1.23 (Pin_23)
- net TDI: now also J1.17 (Pin_17); no longer J1.21 (Pin_21)
- net TDO: now also J1.18 (Pin_18); no longer J1.22 (Pin_22)
- net TMS: now also J1.20 (Pin_20); no longer J1.24 (Pin_24)
- net B_D12: now reaches P1.b10 (10B)
- net B_D12: now also IC1.12 (I/O/PD1)
- net B_D13: now reaches P1.b11 (11B)
- net B_D13: now also IC1.36 (I/O_25)
- net B_D14: now reaches P1.b12 (12B)
- net B_D14: now also IC1.37 (I/O_26)
- net B_D15: now reaches P1.b13 (13B)
- net B_D15: now also IC1.39 (I/O_27)
- net B_ / SXTAK: now reaches P1.b22 (22B)
- net B_ / SXTAK: now also IC1.40 (I/O_28)
- net B_ / SXTRQ: now reaches P1.b24 (24B)
- net B_ / SXTRQ: now also IC1.41 (I/O_29)
- net B_ / DS0: now reaches P1.b28 (28B)
- net B_ / DS0: now also IC1.46 (I/O_31), IC1.48 (I/O_32), P1.b29 (29B)
- net B_D8: now reaches P1.b6 (6B)
- net B_D8: now also IC1.8 (I/O_4)
- net B_D9: now reaches P1.b7 (7B)
- net B_D9: now also IC1.9 (I/O_5)
- net B_D10: now reaches P1.b8 (8B)
- net B_D10: now also IC1.10 (I/O_6)
- net B_D11: now reaches P1.b9 (9B)
- net B_D11: now also IC1.11 (I/O_7)
- removed net IO_25: IC1.36 (I/O_25), J1.16 (Pin_16)
- removed net IO_26: IC1.37 (I/O_26), J1.15 (Pin_15)
- removed net IO_27: IC1.39 (I/O_27), J1.14 (Pin_14)
- removed net IO_28: IC1.40 (I/O_28), J1.13 (Pin_13)
- removed net IO_29: IC1.41 (I/O_29), J1.12 (Pin_12)
- net IO_31: no longer names the net of J1.10 (Pin_10)
- net IO_31: no longer IC1.46 (I/O_31)
- net IO_32: no longer names the net of J1.9 (Pin_9)
- net IO_32: no longer IC1.48 (I/O_32)
- removed net IO_4: IC1.8 (I/O_4), J1.17 (Pin_17)
- removed net IO_5: IC1.9 (I/O_5), J1.18 (Pin_18)
- removed net IO_6: IC1.10 (I/O_6), J1.19 (Pin_19)
- removed net IO_7: IC1.11 (I/O_7), J1.20 (Pin_20)
- net I/O/PD1: no longer names the net of J1.8 (Pin_8)
- net I/O/PD1: no longer IC1.12 (I/O/PD1)
- new net GCLR_FTDI: Q1.1 (G)
- new net RESET_FTDI: Q2.1 (G)
- no-connect marks 48 -> 49
Other:
- sheet JTAG-Interface ports: added GCRL_FTDI, RESET_FTDI; removed none
- moved on the sheet: C2

Commit message: rev 5
Parts:
- removed J1: Conn_02x16_Counter_Clockwise, Connector_PinHeader_2.54mm:PinHeader_2x16_P2.54mm_Vertical, symbol Connector_Generic:Conn_02x16_Counter_Clockwise
- added D3, D4, D5: LED, LED_SMD:LED_0402_1005Metric, symbol Device:LED
- added J2: Conn_02x08_Counter_Clockwise, Connector_PinHeader_2.54mm:PinHeader_2x08_P2.54mm_Vertical, symbol Connector_Generic:Conn_02x08_Counter_Clockwise
- added R12, R13, R14, R3, R4: 5k1, Resistor_SMD:R_0201_0603Metric_Pad0.64x0.40mm_HandSolder, symbol Device:R
- added R5: 0R, Resistor_SMD:R_0201_0603Metric_Pad0.64x0.40mm_HandSolder, symbol Device:R
- R1: renamed from R6; footprint (none) -> Resistor_SMD:R_0201_0603Metric_Pad0.64x0.40mm_HandSolder
- R2: renamed from R8; footprint (none) -> Resistor_SMD:R_0201_0603Metric_Pad0.64x0.40mm_HandSolder
- U1: renamed from IC1; footprint Package_LCC:PLCC-84 -> Package_LCC:PLCC-84_THT-Socket
- renumbered C2 to C1, C10 to C2, C1 to C3, C9 to C4, J2 to J1, U3 to U2, U2 to U3
Connections:
- net IO_30 is gone; now on net B_D12: U1.44 (I/O_30)
- net +3.3V: now also J1.1 (Pin_1), J2.7 (Pin_7)
- net +5V: now also J2.8 (Pin_8); no longer J1.1 (Pin_1)
- net B_ / DS0: no longer P1.b29 (29B), U1.48 (I/O_32)
- net B_D12: no longer U1.12 (I/O/PD1)
- net GCLK1: now also R5.2; no longer U2.5 (OUT)
- net GCLR_FTDI: now also R3.1
- net GND: now also D3.1 (K), D4.1 (K), D5.1 (K), J2.10 (Pin_10), J2.9 (Pin_9), R3.2, R4.2; no longer P1.HOLE (GND)
- net I/GCLR: now also J2.12 (Pin_12)
- net I/OE1: now also J2.11 (Pin_11)
- net I/OE2/GCLK2: now also J2.14 (Pin_14)
- net I/O/GCLK3: now also J2.13 (Pin_13), R14.1
- net I/O/PD2: now also J2.15 (Pin_15), R12.1
- net RESET_FTDI: now also R4.1
- net TCK: now also J2.3 (Pin_3)
- net TDI: now also J2.1 (Pin_1)
- net TDO: now also J2.2 (Pin_2)
- net TMS: now also J2.4 (Pin_4)
- new net: D3.2 (A), R12.2
- new net: R5.1, U2.5 (OUT)
- new net: D5.2 (A), R14.2
- new net: D4.2 (A), R13.2
- new net B_ / DS1: P1.b29 (29B), U1.48 (I/O_32)
- new net I/O/PD1: J2.16 (Pin_16), R13.1, U1.12 (I/O/PD1)
- no-connect marks 49 -> 32
Other:
- sheet JTAG-Interface: file untitled.kicad_sch -> jtag-interface.kicad_sch
- sheet JTAG-Interface ports: added BCBUS0, BCBUS1, BCBUS2, BCBUS3, BCBUS4, GCLR_FTDI; removed GCRL_FTDI
- title: (none) -> Interruptus Dev Board
- moved on the sheet: C3

Commit message: rev 8
Parts:
- removed J2: Conn_02x08_Counter_Clockwise, Connector_PinHeader_2.54mm:PinHeader_2x08_P2.54mm_Vertical, symbol Connector_Generic:Conn_02x08_Counter_Clockwise
- added J4: Conn_02x20_Counter_Clockwise, Connector_PinHeader_2.54mm:PinHeader_2x20_P2.54mm_Vertical, symbol Connector_Generic:Conn_02x20_Counter_Clockwise
- D1: renamed from D3; footprint LED_SMD:LED_0402_1005Metric -> LED_SMD:LED_0603_1608Metric_Pad1.05x0.95mm_HandSolder
- D2: renamed from D4; footprint LED_SMD:LED_0402_1005Metric -> LED_SMD:LED_0603_1608Metric_Pad1.05x0.95mm_HandSolder
- D3: renamed from D5; footprint LED_SMD:LED_0402_1005Metric -> LED_SMD:LED_0603_1608Metric_Pad1.05x0.95mm_HandSolder
- R1, R12, R13, R14, R2, R3, R4, R5: footprint Resistor_SMD:R_0201_0603Metric_Pad0.64x0.40mm_HandSolder -> Resistor_SMD:R_0603_1608Metric_Pad0.98x0.95mm_HandSolder
Connections:
- net +3.3V: now also J4.1 (Pin_1)
- net +5V: now also J4.3 (Pin_3)
- net B_/IRQ0: now also J4.23 (Pin_23)
- net B_/IRQ1: now also J4.24 (Pin_24)
- net B_/IRQ2: now also J4.25 (Pin_25)
- net B_/IRQ3: now also J4.26 (Pin_26)
- net B_/IRQ4: now also J4.27 (Pin_27)
- net B_/RD: now also J4.22 (Pin_22)
- net B_/WR: now also J4.21 (Pin_21)
- net B_A0: now also J4.4 (Pin_4)
- net B_A1: now also J4.5 (Pin_5)
- net B_A2: now also J4.6 (Pin_6)
- net B_A3: now also J4.7 (Pin_7)
- net B_A4: now also J4.8 (Pin_8)
- net B_A5: now also J4.9 (Pin_9)
- net B_A6: now also J4.10 (Pin_10)
- net B_A7: now also J4.11 (Pin_11)
- net B_A8: now also J4.12 (Pin_12)
- net B_D0: now also J4.13 (Pin_13)
- net B_D1: now also J4.14 (Pin_14)
- net B_D2: now also J4.15 (Pin_15)
- net B_D3: now also J4.16 (Pin_16)
- net B_D4: now also J4.17 (Pin_17)
- net B_D5: now also J4.18 (Pin_18)
- net B_D6: now also J4.19 (Pin_19)
- net B_D7: now also J4.20 (Pin_20)
- net B_VCC: now also J4.39 (Pin_39)
- net GND: now also J4.2 (Pin_2), J4.38 (Pin_38), J4.40 (Pin_40)
- net I/GCLR: now also J4.29 (Pin_29)
- net I/OE1: now also J4.28 (Pin_28)
- net I/OE2/GCLK2: now also J4.31 (Pin_31)
- net I/O/GCLK3: now also J4.30 (Pin_30)
- net I/O/PD1: now also J4.33 (Pin_33)
- net I/O/PD2: now also J4.32 (Pin_32)
- net TCK: now also J4.36 (Pin_36)
- net TDI: now also J4.34 (Pin_34)
- net TDO: now also J4.35 (Pin_35)
- net TMS: now also J4.37 (Pin_37)
- no-connect marks 32 -> 30
