File: kicad/interruptus/jtag-interface.kicad_sch (KiCad schematic)
At the start: 15 parts, among them J3 USB4110GFA, U4 FT2232D, Y1 6 MHz

Commit message: rev 5
Parts:
- removed D1, D2: 1N5819, Diode_SMD:Nexperia_CFP3_SOD-123W, symbol Diode:1N5819
- added R15: 2k2, Resistor_SMD:R_0201_0603Metric_Pad0.64x0.40mm_HandSolder, symbol Device:R_Small
- added R16: 10k, Resistor_SMD:R_0201_0603Metric_Pad0.64x0.40mm_HandSolder, symbol Device:R_Small
- added U5: 93CxxB, Package_SO:SOIC-8_3.9x4.9mm_P1.27mm, symbol Memory_EEPROM:93CxxB
- added U6, U7: MAX40200AUK, Package_TO_SOT_SMD:SOT-23-5, symbol Analog_Switch:MAX40200AUK
- J3: footprint Connector_USB:USB_C_Receptacle_GCT_USB4110 -> Library:USB_C_Receptacle_GCT_USB4110
Connections:
- net +5V: now also R16.2, U5.8 (VCC), U6.5 (OUT), U7.5 (OUT)
- net B_VCC: now also U6.1 (VDD)
- net GND: now also J3.A12/B1 (GND), U5.5 (GND), U6.2 (GND), U7.2 (GND); no longer J3.B1/A12 (GND), J3.S2 (GND), J3.S3 (GND), J3.S4 (GND)
- net VBUS: now also J3.A9/B4 (VBUS), U7.1 (VDD); no longer J3.B4/A9 (VBUS)
- net FTDI_USB_DATA-: now reaches R8.1, U4.8 (USBDM)
- net USB_DATA-: now reaches J3.A7 (DN1), J3.B7 (DN2), R8.2
- net USB_DATA+: now reaches J3.A6 (DP1), J3.B6 (DP2), R9.2
- net at U4.1 (EECLK): now also U5.2 (SCLK)
- net at U4.2 (EEDATA): now also R15.1, U5.3 (DI)
- net BCBUS4: now reaches U4.26 (SI/WUB)
- net BCBUS3: now reaches U4.27 (BCBUS3)
- net BCBUS2: now reaches U4.28 (BCBUS2)
- net BCBUS1: now reaches U4.29 (BCBUS1)
- net BCBUS0: now reaches U4.30 (BCBUS0)
- net B_D7: now reaches U4.32 (BDBUS7)
- net B_D6: now reaches U4.33 (BDBUS6)
- net B_D5: now reaches U4.35 (BDBUS5)
- net B_D4: now reaches U4.36 (BDBUS4)
- net B_D3: now reaches U4.37 (BDBUS3)
- net B_D2: now reaches U4.38 (BDBUS2)
- net B_D1: now reaches U4.39 (BDBUS1)
- net B_D0: now reaches U4.40 (BDBUS0)
- net at U4.48 (EECS): now also U5.1 (CS)
- net FTDI_USB_DATA+: now reaches R10.2, R9.1, U4.7 (USBDP)
- new net: R15.2, R16.1, U5.4 (DO)
- no-connect marks 26 -> 12
Other:
- moved on the sheet: R10, R8, R9

Commit message: rev 8
Parts:
- added R17: 10k, Resistor_SMD:R_0603_1608Metric_Pad0.98x0.95mm_HandSolder, symbol Device:R_Small
- R10, R11, R15, R16, R6, R7, R8, R9: footprint Resistor_SMD:R_0201_0603Metric_Pad0.64x0.40mm_HandSolder -> Resistor_SMD:R_0603_1608Metric_Pad0.98x0.95mm_HandSolder
Connections:
- net +5V: now also R17.1; no longer U4.4 (~{RESET})
- net VBUS: now also J3.B4/A9 (VBUS2); no longer J3.A9/B4 (VBUS)
- new net: R17.2, U4.4 (~{RESET})
Changed lines of the file:
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@@
 	(title_block
 		(title "Interruptus Dev Board")
-		(date "2024-06-08")
-		(rev "6")
+		(date "2024-06-15")
+		(rev "8")
 	)
 	(junction
@@
 		)
 	)
+	(wire
+		(pts
+			(xy 106.68 99.06) (xy 114.3 99.06)
+		)
+		(stroke
+			(width 0)
+			(type default)
+		)
+	)
 	(label "VBUS"
 		(at 82.55 74.93 0)
@@
 			)
 		)
-		(property "Footprint" "Resistor_SMD:R_0201_0603Metric_Pad0.64x0.40mm_HandSolder"
+		(property "Footprint" "Resistor_SMD:R_0603_1608Metric_Pad0.98x0.95mm_HandSolder"
 			(at 142.24 45.72 0)
 			(effects
@@
 			)
 		)
-		(property "Footprint" "Resistor_SMD:R_0201_0603Metric_Pad0.64x0.40mm_HandSolder"
+		(property "Footprint" "Resistor_SMD:R_0603_1608Metric_Pad0.98x0.95mm_HandSolder"
 			(at 97.79 85.09 0)
 			(effects
@@
 		(dnp no)
 		(property "Reference" "R16"
-			(at 96.266 148.082 0)
+			(at 96.52 146.304 0)
 			(effects
 				(font
@@
 		)
 		(property "Value" "10k"
-			(at 96.266 145.796 0)
+			(at 96.52 148.336 0)
 			(effects
 				(font
@@
 			)
 		)
-		(property "Footprint" "Resistor_SMD:R_0201_0603Metric_Pad0.64x0.40mm_HandSolder"
+		(property "Footprint" "Resistor_SMD:R_0603_1608Metric_Pad0.98x0.95mm_HandSolder"
 			(at 100.33 146.05 0)
 			(effects
@@
 	(symbol
 		(lib_id "power:+5V")
-		(at 119.38 99.06 90)
+		(at 106.68 99.06 90)
 		(unit 1)
 		(exclude_from_sim no)
@@
 		(fields_autoplaced yes)
 		(property "Reference" "#PWR045"
-			(at 123.19 99.06 0)
+			(at 110.49 99.06 0)
 			(effects
 				(font
@@
 		)
 		(property "Value" "+5V"
-			(at 115.57 99.0599 90)
+			(at 102.87 99.0599 90)
 			(effects
 				(font
@@
 		)
 		(property "Footprint" ""
-			(at 119.38 99.06 0)
+			(at 106.68 99.06 0)
 			(effects
 				(font
@@
 		)
 		(property "Datasheet" ""
-			(at 119.38 99.06 0)
+			(at 106.68 99.06 0)
 			(effects
 				(font
@@
 		)
 		(property "Description" "Power symbol creates a global label with name \"+5V\""
-			(at 119.38 99.06 0)
+			(at 106.68 99.06 0)
 			(effects
 				(font
@@
 			)
 		)
-		(property "Footprint" "Resistor_SMD:R_0201_0603Metric_Pad0.64x0.40mm_HandSolder"
+		(property "Footprint" "Resistor_SMD:R_0603_1608Metric_Pad0.98x0.95mm_HandSolder"
 			(at 92.71 77.47 0)
 			(effects
@@
 		(pin "B6"
 		)
-		(pin "A9/B4"
+		(pin "B4/A9"
 		)
 		(pin "A1/B12"
@@
 			)
 		)
-		(property "Footprint" "Resistor_SMD:R_0201_0603Metric_Pad0.64x0.40mm_HandSolder"
+		(property "Footprint" "Resistor_SMD:R_0603_1608Metric_Pad0.98x0.95mm_HandSolder"
 			(at 97.79 87.63 0)
 			(effects
@@
 			)
 		)
-		(property "Footprint" "Resistor_SMD:R_0201_0603Metric_Pad0.64x0.40mm_HandSolder"
+		(property "Footprint" "Resistor_SMD:R_0603_1608Metric_Pad0.98x0.95mm_HandSolder"
 			(at 125.73 93.98 0)
 			(effects
@@
 			)
 		)
-		(property "Footprint" "Resistor_SMD:R_0201_0603Metric_Pad0.64x0.40mm_HandSolder"
+		(property "Footprint" "Resistor_SMD:R_0603_1608Metric_Pad0.98x0.95mm_HandSolder"
 			(at 105.41 137.16 0)
 			(effects
@@
 	(symbol
 		(lib_id "Device:R_Small")
+		(at 116.84 99.06 90)
+		(unit 1)
+		(exclude_from_sim no)
+		(in_bom yes)
+		(on_board yes)
+		(dnp no)
+		(property "Reference" "R17"
+			(at 117.094 100.838 90)
+			(effects
+				(font
+					(size 1.27 1.27)
+				)
+				(justify bottom)
+			)
+		)
+		(property "Value" "10k"
+			(at 117.094 103.124 90)
+			(effects
+				(font
+					(size 1.27 1.27)
+				)
+				(justify bottom)
+			)
+		)
+		(property "Footprint" "Resistor_SMD:R_0603_1608Metric_Pad0.98x0.95mm_HandSolder"
+			(at 116.84 99.06 0)
+			(effects
+				(font
+					(size 1.27 1.27)
+				)
+				(hide yes)
+			)
+		)
+		(property "Datasheet" "~"
+			(at 116.84 99.06 0)
+			(effects
+				(font
+					(size 1.27 1.27)
+				)
+				(hide yes)
+			)
+		)
+		(property "Description" ""
+			(at 116.84 99.06 0)
+			(effects
+				(font
+					(size 1.27 1.27)
+				)
+				(hide yes)
+			)
+		)
+		(pin "1"
+		)
+		(pin "2"
+		)
+		(instances
+			(project "interruptus"
+				(path "/ee2eecdf-4a5c-4392-b1fa-18b59b455a83/f41f9d35-9a9d-4ed6-b44b-43e12ad79e40"
+					(reference "R17")
+					(unit 1)
+				)
+			)
+		)
+	)
+	(symbol
+		(lib_id "Device:R_Small")
 		(at 34.29 77.47 0)
 		(unit 1)
@@
 			)
 		)
-		(property "Footprint" "Resistor_SMD:R_0201_0603Metric_Pad0.64x0.40mm_HandSolder"
+		(property "Footprint" "Resistor_SMD:R_0603_1608Metric_Pad0.98x0.95mm_HandSolder"
 			(at 34.29 77.47 0)
 			(effects
